File: contrib/aristo-d2-led-panel-v2/led_panel_4x5.kicad_pcb (KiCad board)
At the start: 4 copper layers, 157 x 157 mm, 238 parts, among them U1 C42417599_LED-SMD_4P-L3.5-W3.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, U10 C42417599_LED-SMD_4P-L3.5-W3.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, U100 C42417599_LED-SMD_4P-L3.5-W3.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, U101 C42417599_LED-SMD_4P-L3.5-W3.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, U102 C42417599_LED-SMD_4P-L3.5-W3.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, U103 C42417599_LED-SMD_4P-L3.5-W3.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, U104 C42417599_LED-SMD_4P-L3.5-W3.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, U105 C42417599_LED-SMD_4P-L3.5-W3.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, U106 C42417599_LED-SMD_4P-L3.5-W3.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, U107 C42417599_LED-SMD_4P-L3.5-W3.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, U108 C42417599_LED-SMD_4P-L3.5-W3.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, U109 C42417599_LED-SMD_4P-L3.5-W3.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, U11 C42417599_LED-SMD_4P-L3.5-W3.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, U110 C42417599_LED-SMD_4P-L3.5-W3.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, U111 C42417599_LED-SMD_4P-L3.5-W3.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, U112 C42417599_LED-SMD_4P-L3.5-W3.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, U12 C42417599_LED-SMD_4P-L3.5-W3.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, U13 C42417599_LED-SMD_4P-L3.5-W3.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, U14 C42417599_LED-SMD_4P-L3.5-W3.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, U15 C42417599_LED-SMD_4P-L3.5-W3.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, U16 C42417599_LED-SMD_4P-L3.5-W3.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, U17 C42417599_LED-SMD_4P-L3.5-W3.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, U18 C42417599_LED-SMD_4P-L3.5-W3.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, U19 C42417599_LED-SMD_4P-L3.5-W3.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, U2 C42417599_LED-SMD_4P-L3.5-W3.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, U20 C42417599_LED-SMD_4P-L3.5-W3.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, U21 C42417599_LED-SMD_4P-L3.5-W3.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, U22 C42417599_LED-SMD_4P-L3.5-W3.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, U226 C7484_SOT-23-5_L3.0-W1.7-P0.9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, U23 C42417599_LED-SMD_4P-L3.5-W3.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, U24 C42417599_LED-SMD_4P-L3.5-W3.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, U25 C42417599_LED-SMD_4P-L3.5-W3.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, U26 C42417599_LED-SMD_4P-L3.5-W3.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, U27 C42417599_LED-SMD_4P-L3.5-W3.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, U28 C42417599_LED-SMD_4P-L3.5-W3.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, U29 C42417599_LED-SMD_4P-L3.5-W3.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, U3 C42417599_LED-SMD_4P-L3.5-W3.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, U30 C42417599_LED-SMD_4P-L3.5-W3.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, U31 C42417599_LED-SMD_4P-L3.5-W3.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, U32 C42417599_LED-SMD_4P-L3.5-W3.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, U33 C42417599_LED-SMD_4P-L3.5-W3.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, U34 C42417599_LED-SMD_4P-L3.5-W3.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, U35 C42417599_LED-SMD_4P-L3.5-W3.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, U36 C42417599_LED-SMD_4P-L3.5-W3.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, U37 C42417599_LED-SMD_4P-L3.5-W3.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, U38 C42417599_LED-SMD_4P-L3.5-W3.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, U39 C42417599_LED-SMD_4P-L3.5-W3.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, U4 C42417599_LED-SMD_4P-L3.5-W3.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, U40 C42417599_LED-SMD_4P-L3.5-W3.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, U41 C42417599_LED-SMD_4P-L3.5-W3.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, U42 C42417599_LED-SMD_4P-L3.5-W3.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, U43 C42417599_LED-SMD_4P-L3.5-W3.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, U44 C42417599_LED-SMD_4P-L3.5-W3.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, U45 C42417599_LED-SMD_4P-L3.5-W3.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, U46 C42417599_LED-SMD_4P-L3.5-W3.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, U47 C42417599_LED-SMD_4P-L3.5-W3.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, U48 C42417599_LED-SMD_4P-L3.5-W3.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, U49 C42417599_LED-SMD_4P-L3.5-W3.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, U5 C42417599_LED-SMD_4P-L3.5-W3.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, U50 C42417599_LED-SMD_4P-L3.5-W3.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, U51 C42417599_LED-SMD_4P-L3.5-W3.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, U52 C42417599_LED-SMD_4P-L3.5-W3.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, U53 C42417599_LED-SMD_4P-L3.5-W3.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, U54 C42417599_LED-SMD_4P-L3.5-W3.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, U55 C42417599_LED-SMD_4P-L3.5-W3.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, U56 C42417599_LED-SMD_4P-L3.5-W3.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, U57 C42417599_LED-SMD_4P-L3.5-W3.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, U58 C42417599_LED-SMD_4P-L3.5-W3.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, U59 C42417599_LED-SMD_4P-L3.5-W3.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, U6 C42417599_LED-SMD_4P-L3.5-W3.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, U60 C42417599_LED-SMD_4P-L3.5-W3.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, U61 C42417599_LED-SMD_4P-L3.5-W3.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, U62 C42417599_LED-SMD_4P-L3.5-W3.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, U63 C42417599_LED-SMD_4P-L3.5-W3.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, U64 C42417599_LED-SMD_4P-L3.5-W3.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, U65 C42417599_LED-SMD_4P-L3.5-W3.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, U66 C42417599_LED-SMD_4P-L3.5-W3.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, U67 C42417599_LED-SMD_4P-L3.5-W3.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, U68 C42417599_LED-SMD_4P-L3.5-W3.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, U69 C42417599_LED-SMD_4P-L3.5-W3.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

Commit message: Keep only the back datasheet on the LED panel and refresh the JLCPCB gerbers.
Co-authored-by: Cursor <cursoragent@cursor.com>
Parts:
- moved C212 5.76 mm to (97.3, 65.9)
- moved C211 3.28 mm to (89.0, 65.9)
Routing:
- net 5V: track 428.2 -> 432.3 mm
Other:
- board text added: "Place the fuse next to the 5V pads, not at the PSU."
- board text removed: "Place the fuse next to the 5V pads, not at the power supply."
